File: pcb_kicad/robot_mobilny_pcb/robot_mobilny_pcb.kicad_pcb (KiCad board)
At the start: 2 copper layers, 2 parts, among them J1 Power 14.8V, U1 STM32F411RETx

Commit message: schematic update
Parts:
- added D1: RED2, LED_THT:LED_D5.0mm, F.Cu at (69.0, 114.0)
- added D2: RED, LED_THT:LED_D5.0mm, F.Cu at (69.0, 107.0)
- added D3: LED_G, LED_THT:LED_D5.0mm, F.Cu at (260.4, 52.2)
- added D4: LED_G, LED_THT:LED_D5.0mm, F.Cu at (257.3, 60.8)
- added D5: LED_G, LED_THT:LED_D5.0mm, F.Cu at (264.8, 59.8)
- added D6: LED_Y, LED_THT:LED_D5.0mm, F.Cu at (249.8, 60.8)
- added D7: LED_R, LED_THT:LED_D5.0mm, F.Cu at (267.9, 52.2)
- added J10: UART_WIFI, Connector_Phoenix_MC_HighVoltage:PhoenixContact_MCV_1,5_4-G-5.08_1x04_P5.08mm_Vertical, F.Cu at (38.0, 95.0)
- added J11: LIDAR XH2.54-5P, Connector_JST:JST_EH_B5B-EH-A_1x05_P2.50mm_Vertical, F.Cu at (129.0, 89.0)
- added J12: MOTOR_1&2, Connector_PinHeader_2.54mm:PinHeader_1x13_P2.54mm_Vertical, F.Cu at (66.0, 38.0)
- added J13: ENCODER_MOT_2, Connector_Phoenix_MC_HighVoltage:PhoenixContact_MCV_1,5_4-G-5.08_1x04_P5.08mm_Vertical, F.Cu at (128.0, 43.0)
- added J14: ENCODER_MOT_3, Connector_Phoenix_MC_HighVoltage:PhoenixContact_MCV_1,5_4-G-5.08_1x04_P5.08mm_Vertical, F.Cu at (38.0, 132.0)
- added J15: SWD, Connector_PinHeader_2.54mm:PinHeader_1x04_P2.54mm_Vertical, F.Cu at (281.0, 53.5)
- added J16: MOTOR_3&4, Connector_PinHeader_2.54mm:PinHeader_1x13_P2.54mm_Vertical, F.Cu at (70.9, 133.0)
- added J17: ENCODER_MOT_4, Connector_Phoenix_MC_HighVoltage:PhoenixContact_MCV_1,5_4-G-5.08_1x04_P5.08mm_Vertical, F.Cu at (128.0, 117.0)
- added J18: Conn_01x04_Female, Connector_PinSocket_2.54mm:PinSocket_1x04_P2.54mm_Vertical, F.Cu at (305.2, -9.60)
- added J19: Conn_01x04_Female, Connector_PinSocket_2.54mm:PinSocket_1x04_P2.54mm_Vertical, F.Cu at (324.0, -21.0)
- added J2: TOP_CONN, Connector_PinSocket_2.54mm:PinSocket_1x16_P2.54mm_Vertical, F.Cu at (177.0, -18.0)
- added J20: Conn_01x04_Female, Connector_PinSocket_2.54mm:PinSocket_1x04_P2.54mm_Vertical, F.Cu at (292.0, -3.19)
- added J21: Conn_01x04_Female, Connector_PinSocket_2.54mm:PinSocket_1x04_P2.54mm_Vertical, F.Cu at (305.2, -21.9)
- added J22: Conn_01x04_Female, Connector_PinSocket_2.54mm:PinSocket_1x04_P2.54mm_Vertical, F.Cu at (287.4, -3.19)
- added J23: Conn_01x04_Female, Connector_PinSocket_2.54mm:PinSocket_1x04_P2.54mm_Vertical, F.Cu at (275.0, -2.00)
- added J3: BOOT1, Connector_PinSocket_2.54mm:PinSocket_1x03_P2.54mm_Vertical, F.Cu at (201.0, -21.0)
- added J4: RIGHT_CONN, Connector_PinSocket_2.54mm:PinSocket_1x16_P2.54mm_Vertical, F.Cu at (192.0, -11.0)
- added J5: LEFT_CONN, Connector_PinSocket_2.54mm:PinSocket_1x16_P2.54mm_Vertical, F.Cu at (184.0, -17.0)
- added J6: BOTTOM_CONN, Connector_PinSocket_2.54mm:PinSocket_1x16_P2.54mm_Vertical, F.Cu at (169.2, -21.9)
- added J7: Power 14.8V, Connector_AMASS:AMASS_XT60-M_1x02_P7.20mm_Vertical, F.Cu at (54.8, 131.0)
- added J8: STEP_DOWN_D24V50F5, Connector_PinSocket_2.54mm:PinSocket_1x05_P2.54mm_Vertical, F.Cu at (49.0, 104.8)
- added J9: ENCODER_MOT_1, Connector_Phoenix_MC_HighVoltage:PhoenixContact_MCV_1,5_4-G-5.08_1x04_P5.08mm_Vertical, F.Cu at (38.0, 58.1)
- added JP6: Jumper_3_Bridged12, Connector_PinHeader_2.54mm:PinHeader_1x03_P2.54mm_Vertical, F.Cu at (155.0, 89.9)
- added JP7: ammeter, Connector_PinHeader_2.54mm:PinHeader_1x02_P2.54mm_Vertical, F.Cu at (46.0, 130.5)
- added Q1: IRF540N, Package_TO_SOT_THT:TO-220-3_Vertical, F.Cu at (60.5, 120.0)
- added SW1: RESET, Button_Switch_THT:SW_PUSH_6mm_H9.5mm, F.Cu at (187.3, -22.1)
- added SW3: Button_1, Button_Switch_THT:SW_PUSH_6mm_H9.5mm, F.Cu at (249.4, 50.5)
- added SW4: Button_2, Button_Switch_THT:SW_PUSH_6mm_H9.5mm, F.Cu at (238.8, 59.0)
- added SW5: Button_3, Button_Switch_THT:SW_PUSH_6mm_H9.5mm, F.Cu at (238.0, 32.0)
- added U2: LF33_TO252, Package_TO_SOT_SMD:TO-252-2, F.Cu at (58.0, 108.1)
- J1: value Power 14.8V -> BOOT0; footprint Connector_AMASS:AMASS_XT60-M_1x02_P7.20mm_Vertical -> Connector_PinSocket_2.54mm:PinSocket_1x03_P2.54mm_Vertical
- moved U1 106.9 mm to (84.0, 83.0), turned to 45 degrees
Connections:
- J1 pad 1: (no net) -> +3V3
- U1 pad 1: (no net) -> +3V3
- U1 pad 12: (no net) -> +3V3
- U1 pad 13: (no net) -> +3V3
- U1 pad 14: (no net) -> M1PWM
- U1 pad 15: (no net) -> M2PWM
- U1 pad 16: (no net) -> M3PWM
- U1 pad 17: (no net) -> M4PWM
- U1 pad 18: GND -> +3V3
- U1 pad 19: (no net) -> +3V3
- U1 pad 2: (no net) -> BUTTON_2
- U1 pad 21: (no net) -> ENCODER_2_A
- U1 pad 25: (no net) -> LED5
- U1 pad 29: (no net) -> M1INB
- U1 pad 31: GND -> +3V3
- U1 pad 32: (no net) -> +3V3
- U1 pad 33: (no net) -> M2INA
- U1 pad 34: (no net) -> M2INB
- U1 pad 35: (no net) -> M3INA
- U1 pad 36: (no net) -> M3INB
- U1 pad 37: (no net) -> ENCODER_3_A
- U1 pad 38: (no net) -> ENCODER_3_B
- U1 pad 39: (no net) -> LED1
- U1 pad 40: (no net) -> LED2
- U1 pad 41: (no net) -> ENCODER_1_A
- U1 pad 42: (no net) -> ENCODER_1_B
- U1 pad 43: (no net) -> UART1_RX
- U1 pad 44: (no net) -> UART6_TX
- U1 pad 45: (no net) -> UART6_RX
- U1 pad 46: (no net) -> SWDIO
- U1 pad 47: GND -> +3V3
- U1 pad 48: (no net) -> +3V3
- U1 pad 49: (no net) -> SWCLK
- U1 pad 50: (no net) -> UART1_TX
- U1 pad 51: (no net) -> LED3
- U1 pad 52: (no net) -> LED4
- U1 pad 53: (no net) -> BUTTON_1
- U1 pad 55: (no net) -> ENCODER_2_B
- U1 pad 56: (no net) -> M4INA
- U1 pad 57: (no net) -> M4INB
- U1 pad 58: (no net) -> ENCODER_4_A
- U1 pad 59: (no net) -> ENCODER_4_B
- U1 pad 61: (no net) -> PWM_LIDAR
- U1 pad 62: (no net) -> M1INA
- U1 pad 63: GND -> +3V3
- U1 pad 64: (no net) -> +3V3
- U1 pad 7: (no net) -> Net-(C1-Pad1)
- U1 pad 9: (no net) -> BUTTON_3
Other:
- board text added: "FRONT"
- board text added: "LEFT"
- board text added: "RIGHT"

Commit message: schematic_update
Parts:
- removed the D2 at (69.0, 107.0)
- removed D7: LED_R, LED_THT:LED_D5.0mm
- removed J15: SWD, Connector_PinHeader_2.54mm:PinHeader_1x04_P2.54mm_Vertical
- removed J16: MOTOR_3&4, Connector_PinHeader_2.54mm:PinHeader_1x13_P2.54mm_Vertical
- removed J23: Conn_01x04_Female, Connector_PinSocket_2.54mm:PinSocket_1x04_P2.54mm_Vertical
- removed J4: RIGHT_CONN, Connector_PinSocket_2.54mm:PinSocket_1x16_P2.54mm_Vertical
- removed J5: LEFT_CONN, Connector_PinSocket_2.54mm:PinSocket_1x16_P2.54mm_Vertical
- removed J6: BOTTOM_CONN, Connector_PinSocket_2.54mm:PinSocket_1x16_P2.54mm_Vertical
- removed J8: STEP_DOWN_D24V50F5, Connector_PinSocket_2.54mm:PinSocket_1x05_P2.54mm_Vertical
- removed JP6: Jumper_3_Bridged12, Connector_PinHeader_2.54mm:PinHeader_1x03_P2.54mm_Vertical
- removed JP7: ammeter, Connector_PinHeader_2.54mm:PinHeader_1x02_P2.54mm_Vertical
- removed SW3: Button_1, Button_Switch_THT:SW_PUSH_6mm_H9.5mm
- removed U2: LF33_TO252, Package_TO_SOT_SMD:TO-252-2
- added BZ201: Buzzer, Buzzer_Beeper:Buzzer_12x9.5RM7.6, F.Cu at (110.5, 124.8)
- added C1: 100nF, Capacitor_THT:C_Disc_D5.0mm_W2.5mm_P2.50mm, F.Cu at (73.2, 78.8)
- added C101: 100nF, Capacitor_THT:C_Disc_D5.0mm_W2.5mm_P2.50mm, F.Cu at (42.0, 101.0)
- added C2: 100nF, Capacitor_THT:C_Disc_D5.0mm_W2.5mm_P2.50mm, F.Cu at (90.2, 78.8)
- added C201: 100nF, Capacitor_THT:C_Disc_D5.0mm_W2.5mm_P2.50mm, F.Cu at (95.5, 138.8)
- added C202: 100nF, Capacitor_THT:C_Disc_D5.0mm_W2.5mm_P2.50mm, F.Cu at (105.2, 138.8)
- added C203: 100nF, Capacitor_THT:C_Disc_D5.0mm_W2.5mm_P2.50mm, F.Cu at (115.0, 138.8)
- added C3: 100nF, Capacitor_THT:C_Disc_D5.0mm_W2.5mm_P2.50mm, F.Cu at (92.8, 93.2)
- added C4: 100nF, Capacitor_THT:C_Disc_D5.0mm_W2.5mm_P2.50mm, F.Cu at (73.2, 93.2)
- added C5: 100nF, Capacitor_THT:C_Disc_D5.0mm_W2.5mm_P2.50mm, F.Cu at (55.8, 122.8)
- added C6: 2,2uF, Capacitor_THT:CP_Radial_D4.0mm_P1.50mm, F.Cu at (69.0, 127.5)
- added D1: RED, LED_THT:LED_D5.0mm, F.Cu at (70.5, 142.0)
- added J307: SWD, Connector_PinHeader_2.54mm:PinHeader_1x04_P2.54mm_Vertical, F.Cu at (154.0, 95.4)
- added J308: LSM303D_acc+mag, Connector_PinSocket_2.54mm:PinSocket_1x09_P2.54mm_Vertical, F.Cu at (116.2, 27.5)
- added J309: MOTOR_3&4, Connector_PinHeader_2.54mm:PinHeader_1x13_P2.54mm_Vertical, F.Cu at (69.8, 187.8)
- added J315: Conn_01x04_Female, Connector_PinSocket_2.54mm:PinSocket_1x04_P2.54mm_Vertical, F.Cu at (371.5, 2.75)
- added J401: TOP_CONN, Connector_PinSocket_2.54mm:PinSocket_1x16_P2.54mm_Vertical, F.Cu at (64.1, 62.5)
- added J402: RIGHT_CONN, Connector_PinSocket_2.54mm:PinSocket_1x16_P2.54mm_Vertical, F.Cu at (106.5, 66.7)
- added J403: LEFT_CONN, Connector_PinSocket_2.54mm:PinSocket_1x16_P2.54mm_Vertical, F.Cu at (59.8, 105.0)
- added J404: BOTTOM_CONN, Connector_PinSocket_2.54mm:PinSocket_1x16_P2.54mm_Vertical, F.Cu at (102.0, 109.5)
- added JP1: ammeter, Connector_PinHeader_2.54mm:PinHeader_1x02_P2.54mm_Vertical, F.Cu at (47.8, 141.8)
- added JP101: Jumper_3_Bridged12, Connector_PinHeader_2.54mm:PinHeader_1x03_P2.54mm_Vertical, F.Cu at (330.7, 167.6)
- added JP102: Jumper_3_Bridged12, Connector_PinHeader_2.54mm:PinHeader_1x03_P2.54mm_Vertical, F.Cu at (326.1, 167.6)
- added JP103: Jumper_3_Bridged12, Connector_PinHeader_2.54mm:PinHeader_1x03_P2.54mm_Vertical, F.Cu at (330.9, 157.9)
- added JP104: Jumper_3_Bridged12, Connector_PinHeader_2.54mm:PinHeader_1x03_P2.54mm_Vertical, F.Cu at (326.2, 157.9)
- added JP105: Jumper_3_Bridged12, Connector_PinHeader_2.54mm:PinHeader_1x03_P2.54mm_Vertical, F.Cu at (321.6, 158.0)
- added JP106: Jumper_3_Bridged12, Connector_PinHeader_2.54mm:PinHeader_1x03_P2.54mm_Vertical, F.Cu at (321.4, 167.6)
- added JP107: Jumper_3_Bridged12, Connector_PinHeader_2.54mm:PinHeader_1x03_P2.54mm_Vertical, F.Cu at (263.0, 163.0)
- added JP108: Jumper_3_Bridged12, Connector_PinHeader_2.54mm:PinHeader_1x03_P2.54mm_Vertical, F.Cu at (276.0, 163.0)
- added R1: 100k, Resistor_THT:R_Axial_DIN0207_L6.3mm_D2.5mm_P10.16mm_Horizontal, F.Cu at (47.5, 132.8)
- added R101: 10k, Resistor_THT:R_Axial_DIN0207_L6.3mm_D2.5mm_P10.16mm_Horizontal, F.Cu at (45.0, 101.0)
- added R102: 10k, Resistor_THT:R_Axial_DIN0207_L6.3mm_D2.5mm_P10.16mm_Horizontal, F.Cu at (48.5, 68.0)
- added R105: 10k, Resistor_THT:R_Axial_DIN0207_L6.3mm_D2.5mm_P10.16mm_Horizontal, F.Cu at (111.8, 80.8)
- added R201: 330, Resistor_THT:R_Axial_DIN0207_L6.3mm_D2.5mm_P10.16mm_Horizontal, F.Cu at (72.0, 41.8)
- added R202: 330, Resistor_THT:R_Axial_DIN0207_L6.3mm_D2.5mm_P10.16mm_Horizontal, F.Cu at (109.0, 105.0)
- added R203: 4k7, Resistor_THT:R_Axial_DIN0207_L6.3mm_D2.5mm_P10.16mm_Horizontal, F.Cu at (98.8, 131.6)
- added R204: 330, Resistor_THT:R_Axial_DIN0207_L6.3mm_D2.5mm_P10.16mm_Horizontal, F.Cu at (78.8, 41.8)
- added R205: 330, Resistor_THT:R_Axial_DIN0207_L6.3mm_D2.5mm_P10.16mm_Horizontal, F.Cu at (85.5, 41.8)
- added R206: 330, Resistor_THT:R_Axial_DIN0207_L6.3mm_D2.5mm_P10.16mm_Horizontal, F.Cu at (92.2, 41.8)
- added R207: 4k7, Resistor_THT:R_Axial_DIN0207_L6.3mm_D2.5mm_P10.16mm_Horizontal, F.Cu at (108.5, 131.5)
- added R208: 4k7, Resistor_THT:R_Axial_DIN0207_L6.3mm_D2.5mm_P10.16mm_Horizontal, F.Cu at (118.2, 131.5)
- added R3: 470, Resistor_THT:R_Axial_DIN0207_L6.3mm_D2.5mm_P10.16mm_Horizontal, F.Cu at (75.5, 132.0)
- added R4: 470, Resistor_THT:R_Axial_DIN0207_L6.3mm_D2.5mm_P10.16mm_Horizontal, F.Cu at (78.5, 132.0)
- added R5: 47k, Resistor_THT:R_Axial_DIN0207_L6.3mm_D2.5mm_P10.16mm_Horizontal, F.Cu at (64.8, 133.8)
- added SW101: RESET, Button_Switch_THT:SW_PUSH_6mm_H9.5mm, F.Cu at (35.3, 104.0)
- added SW201: Button_1, Button_Switch_THT:SW_PUSH_6mm_H9.5mm, F.Cu at (98.8, 144.5)
- added U1: LF33_TO252, Package_TO_SOT_SMD:TO-252-2, F.Cu at (61.8, 125.8)
- added Y101: 8Mhz, Crystal:Crystal_HC49-4H_Vertical, F.Cu at (276.0, 155.0)
- added Y102: Crystal, Crystal:Crystal_HC49-4H_Vertical, F.Cu at (260.0, 154.0)
- J101: renamed from J1; footprint Connector_PinSocket_2.54mm:PinSocket_1x03_P2.54mm_Vertical -> Connector_PinHeader_2.54mm:PinHeader_1x03_P2.54mm_Vertical
- J102: renamed from J3; footprint Connector_PinSocket_2.54mm:PinSocket_1x03_P2.54mm_Vertical -> Connector_PinHeader_2.54mm:PinHeader_1x03_P2.54mm_Vertical
- J2: value TOP_CONN -> STEP_DOWN_D24V50F5; footprint Connector_PinSocket_2.54mm:PinSocket_1x16_P2.54mm_Vertical -> Connector_PinSocket_2.54mm:PinSocket_1x05_P2.54mm_Vertical
- J311: renamed from J18; footprint Connector_PinSocket_2.54mm:PinSocket_1x04_P2.54mm_Vertical -> Connector_PinHeader_2.54mm:PinHeader_1x04_P2.54mm_Vertical
- SW1: value RESET -> SW_SPDT; footprint Button_Switch_THT:SW_PUSH_6mm_H9.5mm -> Button_Switch_THT:SW_CuK_JS202011CQN_DPDT_Straight
- moved SW1 216.8 mm to (50.8, 146.2), turned to 270 degrees
- moved J2 199.7 mm to (50.8, 136.8), turned to 180 degrees
- moved D201 188.4 mm to (72.0, 47.5), turned to 90 degrees
- moved D203 179.7 mm to (85.5, 47.5), turned to 90 degrees
- moved D202 179.1 mm to (78.8, 47.5), turned to 90 degrees
- moved SW203 164.3 mm to (118.2, 144.5), turned to 270 degrees
- moved D204 158.1 mm to (92.2, 47.5), turned to 90 degrees
- moved SW202 155.9 mm to (108.5, 144.6), turned to 270 degrees
- moved J102 136.1 mm to (116.5, 85.8)
- moved J101 113.8 mm to (49.0, 72.2), turned to 270 degrees
- moved D2 21.1 mm to (70.5, 135.0)
- moved J304 19.2 mm to (66.0, 18.8)
- moved J1 18.0 mm to (57.5, 148.8)
- moved Q1 18.0 mm to (63.3, 137.8)
- moved J311 13.4 mm to (311.5, 2.25)
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- renumbered D1 to D2, D3 to D201, D4 to D202, D5 to D203, D6 to D204, J7 to J1, J9 to J301, J10 to J302, J11 to J303, J12 to J304, J13 to J305, J14 to J306, J17 to J310, J19 to J312, J20 to J313, J21 to J314, J22 to J316, SW4 to SW202, SW5 to SW203, U1 to U101
Connections:
- D2 pad 1: (no net) -> Net-(D2-Pad1)
- D201 pad 2: (no net) -> Net-(D201-Pad2)
- D202 pad 2: (no net) -> Net-(D202-Pad2)
- D203 pad 2: (no net) -> Net-(D203-Pad2)
- D204 pad 2: (no net) -> Net-(D204-Pad2)
- J1 pad 1: (no net) -> Net-(J1-Pad1)
- J101 pad 1: +3V3 -> GND
- J101 pad 2: (no net) -> Net-(J101-Pad2)
- J102 pad 2: (no net) -> Net-(J102-Pad2)
- J102 pad 3: +3V3 -> GND
- J2 pad 2: (no net) -> +BATT
- J2 pad 3: (no net) -> GND
- J2 pad 4: (no net) -> GND
- J2 pad 5: (no net) -> +5V
- J301 pad 4: +3V3 -> GND
- J302 pad 4: +3V3 -> GND
- J303 pad 2: +3V3 -> GND
- J304 pad 1: +3V3 -> GND
- J304 pad 4: (no net) -> +3V3
- J304 pad 9: (no net) -> +3V3
- J305 pad 4: +3V3 -> GND
- J306 pad 4: +3V3 -> GND
- J310 pad 4: +3V3 -> GND
- J311 pad 1: +3V3 -> GND
- J311 pad 2: (no net) -> Dist_Sens_01_Echo
- J311 pad 3: (no net) -> Dist_Sens_01_Trig
- J312 pad 1: +3V3 -> GND
- J312 pad 2: (no net) -> Dist_Sens_02_Echo
- J312 pad 3: (no net) -> Dist_Sens_02_Trig
- J313 pad 1: +3V3 -> GND
- J313 pad 2: (no net) -> Dist_Sens_03_Echo
- J313 pad 3: (no net) -> Dist_Sens_03_Trig
- J314 pad 1: +3V3 -> GND
- J314 pad 2: (no net) -> Dist_Sens_04_Echo
- J314 pad 3: (no net) -> Dist_Sens_04_Trig
- J316 pad 1: +3V3 -> GND
- J316 pad 2: (no net) -> Dist_Sens_05_Echo
- J316 pad 3: (no net) -> Dist_Sens_05_Trig
- Q1 pad 1: (no net) -> Net-(Q1-Pad1)
- Q1 pad 3: +3V3 -> GND
- SW1 pad 1: Net-(C1-Pad1) -> (no net)
- SW1 pad 2: +3V3 -> Net-(J1-Pad1)
- SW202 pad 2: +3V3 -> GND
- SW203 pad 2: +3V3 -> GND
- U101 pad 10: (no net) -> M1INB
- U101 pad 11: (no net) -> M1INA
- U101 pad 12: +3V3 -> GND
- U101 pad 18: +3V3 -> GND
- U101 pad 20: (no net) -> ADC_BAT
- U101 pad 22: (no net) -> Dist_Sens_01_Echo
- U101 pad 23: (no net) -> Dist_Sens_01_Trig
- U101 pad 24: (no net) -> BUZZER
- U101 pad 25: LED5 -> BUTTON_3
- U101 pad 26: (no net) -> Dist_Sens_02_Trig
- U101 pad 27: (no net) -> Dist_Sens_02_Echo
- U101 pad 28: (no net) -> Net-(JP105-Pad2)
- U101 pad 29: M1INB -> I2C2_SCL_mag+acc
- U101 pad 3: (no net) -> Net-(JP106-Pad2)
- U101 pad 31: +3V3 -> GND
- U101 pad 4: (no net) -> Net-(JP108-Pad2)
- U101 pad 44: UART6_TX -> Net-(JP102-Pad2)
- U101 pad 45: UART6_RX -> Net-(JP104-Pad2)
- U101 pad 47: +3V3 -> GND
- U101 pad 5: (no net) -> Net-(JP101-Pad2)
- U101 pad 54: (no net) -> PD2
- U101 pad 6: (no net) -> Net-(JP103-Pad2)
- U101 pad 60: (no net) -> BOOT0
- U101 pad 61: PWM_LIDAR -> Net-(JP107-Pad2)
- U101 pad 62: M1INA -> I2C2_SDA_mag+acc
- U101 pad 63: +3V3 -> GND
- U101 pad 7: Net-(C1-Pad1) -> NRST
- U101 pad 8: (no net) -> Dist_Sens_05_Echo
- U101 pad 9: BUTTON_3 -> Dist_Sens_05_Trig
Routing:
- net +5V: track 0.00 -> 19.1 mm
- net Net-(JP1-Pad1): track 0.00 -> 17.1 mm
- net +BATT: track 0.00 -> 13.4 mm
- net Net-(D1-Pad1): track 0.00 -> 13.3 mm
- net Net-(J1-Pad2): track 0.00 -> 12.7 mm
- net Net-(J1-Pad1): track 0.00 -> 6.80 mm
- net Net-(Q1-Pad1): track 0.00 -> 4.60 mm
Other:
- net class Motor added: clearance 0.2, trace_width 1, via_dia 0.8, via_drill 0.4
- net class POWER added: clearance 0.2, trace_width 1.5, via_dia 0.8, via_drill 0.4

Commit message: PCB_update
Change of  motor controller connector to Arduino shields
Parts:
- removed J304: MOTOR_1&2, Connector_PinHeader_2.54mm:PinHeader_1x13_P2.54mm_Vertical
- removed J309: MOTOR_3&4, Connector_PinHeader_2.54mm:PinHeader_1x13_P2.54mm_Vertical
- removed JP101, JP102, JP103, JP106, JP108: Jumper_3_Bridged12, Connector_PinHeader_2.54mm:PinHeader_1x03_P2.54mm_Vertical
- removed Y101: 8Mhz, Crystal:Crystal_HC49-4H_Vertical
- removed Y102: Crystal, Crystal:Crystal_HC49-4H_Vertical
- added A1: Arduino_UNO_R3, Module:Arduino_UNO_R3, F.Cu at (60.2, 188.0)
- added A2: Arduino_UNO_R3, Module:Arduino_UNO_R3, F.Cu at (118.8, 139.8)
- added C102: 4.7uF, Capacitor_THT:C_Disc_D5.0mm_W2.5mm_P2.50mm, F.Cu at (92.0, 73.0)
- added J3: Motor Driver Power, TerminalBlock_Phoenix:TerminalBlock_Phoenix_MKDS-1,5-4_1x04_P5.00mm_Horizontal, F.Cu at (36.2, 132.0)
- added R2: 10k, Resistor_THT:R_Axial_DIN0207_L6.3mm_D2.5mm_P10.16mm_Horizontal, F.Cu at (35.8, 102.8)
- added R6: 10k, Resistor_THT:R_Axial_DIN0207_L6.3mm_D2.5mm_P10.16mm_Horizontal, F.Cu at (38.8, 112.9)
- added UART6/Sens6: Jumper_3_Bridged12, Connector_PinHeader_2.54mm:PinHeader_1x03_P2.54mm_Vertical, F.Cu at (121.2, 54.5)
- J312: footprint Connector_PinSocket_2.54mm:PinSocket_1x04_P2.54mm_Vertical -> Connector_PinHeader_2.54mm:PinHeader_1x04_P2.54mm_Vertical
- SW1: value SW_SPDT -> SWITCH
- moved J311 340.5 mm to (17.0, 173.1)
- moved J312 315.5 mm to (93.1, 194.0), turned to 270 degrees
- moved J314 298.5 mm to (17.8, 58.5)
- moved J315 287.3 mm to (85.5, 30.0), turned to 90 degrees
- moved JP104 231.3 mm to (121.2, 50.8), turned to 90 degrees
- moved JP105 230.3 mm to (99.2, 98.0), turned to 180 degrees
- moved J313 216.2 mm to (161.8, 173.0)
- moved JP107 210.8 mm to (85.0, 50.0), turned to 180 degrees
- moved J316 135.8 mm to (161.0, 58.5)
- moved R201 76.2 mm to (130.8, 90.2), turned to 180 degrees
- moved D201 70.4 mm to (122.8, 96.2)
- moved D202 70.4 mm to (129.5, 96.2)
- moved D203 70.4 mm to (136.2, 96.2)
- moved D204 70.4 mm to (143.0, 96.2)
- moved R205 69.3 mm to (135.0, 90.2), turned to 0 degrees
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Connections:
- Q1 pad 2: Net-(J1-Pad2) -> Net-(J1-Pad1)
- SW1 pad 2: Net-(J1-Pad1) -> Net-(J1-Pad2)
- U101 pad 3: Net-(JP106-Pad2) -> Dist_Sens_04_Trig
- U101 pad 30: (no net) -> Net-(C102-Pad1)
- U101 pad 4: Net-(JP108-Pad2) -> Dist_Sens_04_Echo
- U101 pad 5: Net-(JP101-Pad2) -> INT1_mag+acc
- U101 pad 6: Net-(JP103-Pad2) -> INT2_mag+acc
Routing:
- net NRST: track 0.00 -> 26.9 mm
- net +5V: track 19.1 -> 0.00 mm
- net Net-(JP1-Pad1): track 17.1 -> 0.00 mm
- net BUTTON_1: track 0.00 -> 13.9 mm
- net +BATT: track 13.4 -> 0.00 mm
- net Net-(D1-Pad1): track 13.3 -> 0.00 mm
- net BUTTON_2: track 0.00 -> 12.8 mm
- net BUTTON_3: track 0.00 -> 12.8 mm
- net Net-(J1-Pad2): track 12.7 -> 0.00 mm
- net Net-(D204-Pad2): track 0.00 -> 10.7 mm
- net Net-(D201-Pad2): track 0.00 -> 9.43 mm
- net Net-(D202-Pad2): track 0.00 -> 7.91 mm
- net Net-(J1-Pad1): track 6.80 -> 0.00 mm
- net ADC_BAT: track 0.00 -> 4.75 mm
- net Net-(Q1-Pad1): track 4.60 -> 0.00 mm
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Other:
- board outline added: 150 x 170 mm
- copper layers 2 -> 4

Commit message: PCB_update
Parts:
- removed JP1: ammeter, Connector_PinHeader_2.54mm:PinHeader_1x02_P2.54mm_Vertical
- added J4: Motor Driver Power_not_reverse, TerminalBlock_Phoenix:TerminalBlock_Phoenix_MKDS-1,5-4_1x04_P5.00mm_Horizontal, F.Cu at (36.4, 192.0)
- SW1: footprint Button_Switch_THT:SW_CuK_JS202011CQN_DPDT_Straight -> my_footprint:Button_MRS-101
- moved C201 67.2 mm to (116.2, 181.0)
- moved C202 67.2 mm to (127.2, 181.0)
- moved C203 67.2 mm to (137.0, 181.0)
- moved R203 67.2 mm to (120.8, 174.0)
- moved R207 67.2 mm to (130.5, 173.8)
- moved R208 67.2 mm to (140.2, 173.8)
- moved SW201 67.2 mm to (120.8, 186.8)
- moved SW202 67.2 mm to (130.4, 186.8)
- moved SW203 67.2 mm to (140.2, 186.8)
- moved J3 63.7 mm to (57.6, 192.0), turned to 0 degrees
- moved C5 61.5 mm to (61.8, 164.8)
- moved C6 61.5 mm to (73.5, 164.0)
- moved D1 61.5 mm to (65.2, 175.2)
- moved D2 61.5 mm to (71.8, 175.2)
- moved J2 61.5 mm to (50.2, 177.0)
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- renumbered UART6/Sens6 to JP102
Connections:
- C102 pad 1: Net-(C102-Pad1) -> VCAP_1
- J401 pad 2: +3V3 -> GND
- J401 pad 4: PWM_LIDAR -> PB9
- J402 pad 13: UART1_TX -> M3INB
- J402 pad 14: SWCLK -> M3INA
- J402 pad 15: SWDIO -> M2INB
- J402 pad 2: +3V3 -> GND
- J402 pad 4: UART6_RX -> PA12
- J402 pad 5: UART6_TX -> PA11
- J403 pad 16: (no net) -> +3V3
- J403 pad 5: +3V3 -> GND
- J404 pad 1: Net-(J404-Pad1) -> +3V3
- J404 pad 14: Net-(J404-Pad14) -> +3V3
- J404 pad 15: Net-(J404-Pad14) -> GND
- J404 pad 2: Net-(J404-Pad1) -> GND
- J404 pad 3: (no net) -> VCAP_1
- J404 pad 5: Dist_Sens_03_Trig -> PB2
- JP102 pad 2: Net-(JP102-Pad2) -> PA11
- JP104 pad 2: Net-(JP104-Pad2) -> PA12
- JP105 pad 2: Net-(JP105-Pad2) -> PB2
- JP107 pad 2: Net-(JP107-Pad2) -> PB9
- SW1 pad 3: Net-(JP1-Pad1) -> +BATT
- U101 pad 28: Net-(JP105-Pad2) -> PB2
- U101 pad 30: Net-(C102-Pad1) -> VCAP_1
- U101 pad 44: Net-(JP102-Pad2) -> PA11
- U101 pad 45: Net-(JP104-Pad2) -> PA12
- U101 pad 61: Net-(JP107-Pad2) -> PB9
Routing:
- net +5V: track 0.00 -> 658.5 mm
- net +3V3: track 0.00 -> 416.9 mm
- net ENCODER_3_B: track 0.00 -> 235.7 mm, vias 0 -> 3
- net ENCODER_3_A: track 0.00 -> 228.8 mm, vias 0 -> 3
- net Dist_Sens_03_Echo: track 0.00 -> 217.0 mm, vias 0 -> 2
- net ENCODER_4_B: track 0.00 -> 216.5 mm, vias 0 -> 1
- net BUTTON_2: track 12.8 -> 225.8 mm, vias 0 -> 2
- net ENCODER_4_A: track 0.00 -> 206.1 mm, vias 0 -> 1
- net M1INB: track 0.00 -> 191.6 mm, vias 0 -> 1
- net M1PWM: track 0.00 -> 190.9 mm, vias 0 -> 1
- net M1INA: track 0.00 -> 189.8 mm, vias 0 -> 1
- net ENCODER_2_A: track 0.00 -> 180.7 mm, vias 0 -> 4
- net BUTTON_1: track 13.9 -> 187.3 mm
- net Dist_Sens_01_Trig: track 0.00 -> 166.3 mm, vias 0 -> 3
- net M2PWM: track 0.00 -> 164.5 mm, vias 0 -> 2
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- added copper zone on F.Cu, net +3V3
- added copper zone on B.Cu, net GND
Other:
- net class POWER: trace_width 1.5 -> 3.5
