File: pcb_kicad_2/robot_mobilny_pcb/robot_mobilny_pcb.sch (KiCad schematic (older format))
At the start: 13 parts, among them J101 BOOT0, J102 BOOT1, SW101 RESET, U101 STM32F411RETx

Commit message: pcb v2
version 2 (shorter)
Changed lines of the file:
@@
 	4600 5450 4600 5350
 $Sheet
-S 9450 2400 950  500
+S 8950 2400 950  500
 U 61770FA2
 F0 "interface" 50
@@
 $EndComp
 $Sheet
-S 9450 3250 950  500
+S 8950 3250 950  500
 U 617D3880
 F0 "shields" 50
@@
 	5300 2450 5400 2450
 $Sheet
-S 9450 1450 950  500
+S 8950 1450 950  500
 U 61720EC8
 F0 "power_section" 50
