File: pcb_kicad_2/robot_mobilny_pcb/robot_mobilny_pcb.kicad_pcb (KiCad board)
At the start: 4 copper layers, 150 x 170 mm, 73 parts, among them J1 Power 14.8V, J101 BOOT0, J102 BOOT1, J2 STEP_DOWN_D24V50F5, J3 Motor Driver Power, J301 ENCODER_MOT_1, J302 UART_WIFI, J303 LIDAR XH2.54-5P, J305 ENCODER_MOT_2, J306 ENCODER_MOT_3, J307 SWD, J308 LSM303D_acc+mag, J310 ENCODER_MOT_4, J311 Conn_01x04_Female, J312 Conn_01x04_Female, J313 Conn_01x04_Female, J314 Conn_01x04_Female, J315 Conn_01x04_Female, J316 Conn_01x04_Female, J4 Motor Driver Power_not_reverse, Q1 IRF540N, SW1 SWITCH, SW101 RESET, SW201 Button_1, SW202 Button_2, SW203 Button_3, U1 LF33_TO252, U101 STM32F411RETx

Commit message: pcb v2
version 2 (shorter)
Parts:
- moved C102 3.01 mm to (96.0, 140.0), turned to 0 degrees
- moved C2 1.46 mm to (96.4, 123.8)
- moved A1 0.11 mm to (60.0, 152.4)
Routing:
- net Dist_Sens_05_Echo: track 0.00 -> 120.0 mm, vias 0 -> 2
- net Dist_Sens_05_Trig: track 0.00 -> 117.3 mm, vias 0 -> 2
- net ENCODER_2_A: track 0.00 -> 114.7 mm, vias 0 -> 4
- net ENCODER_2_B: track 0.00 -> 112.9 mm, vias 0 -> 2
- net INT2_mag+acc: track 0.00 -> 106.1 mm, vias 0 -> 2
- net INT1_mag+acc: track 0.00 -> 103.8 mm, vias 0 -> 2
- net M1INB: track 9.04 -> 110.9 mm, vias 0 -> 10
- net I2C2_SCL_mag+acc: track 0.00 -> 95.8 mm, vias 0 -> 4
- net I2C2_SDA_mag+acc: track 0.00 -> 95.8 mm, vias 0 -> 6
- net M1INA: track 13.4 -> 108.2 mm, vias 0 -> 10
- net PB2: track 0.00 -> 90.9 mm, vias 0 -> 10
- net BUTTON_2: track 61.8 -> 129.1 mm, vias 0 -> 4
- net M4INA: track 0.00 -> 66.9 mm, vias 0 -> 4
- net M4INB: track 0.00 -> 65.5 mm, vias 0 -> 2
- net SWDIO: track 0.00 -> 65.0 mm, vias 0 -> 6
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- added copper zone on F.Cu, net GND
Other:
- board size 150 x 170 mm -> 150 x 142.2 mm
- rule trace_min: 0.2 -> 0.25

Commit message: pcb
Parts:
- JP104: value Jumper_3_Bridged12 -> Zwora
- moved A1 0.19 mm to (59.8, 152.5)
- moved C3 0.10 mm to (96.0, 136.9)
- renumbered SW101 to RESET
Routing:
- net +BATT: track 131.2 -> 164.4 mm
- net UART1_TX: track 81.3 -> 97.1 mm, vias 0 -> 6
- net PB2: track 90.9 -> 80.7 mm
- net PA11: track 55.9 -> 62.2 mm, vias 4 -> 6
- net UART1_RX: track 114.8 -> 110.7 mm, vias 6 -> 3
- net SWCLK: track 57.4 -> 60.6 mm
- net PB9: track 105.8 -> 108.6 mm
- net ENCODER_4_B: track 134.5 -> 136.8 mm
- net ENCODER_3_B: track 126.9 -> 129.1 mm, vias 5 -> 6
- net SWDIO: track 65.0 -> 66.9 mm
- net ENCODER_2_B: track 112.9 -> 114.7 mm
- net LED2: track 67.3 -> 65.8 mm
- net PA12: track 62.1 -> 63.5 mm
- net ENCODER_4_A: track 124.2 -> 125.6 mm
- net +3V3: track 486.0 -> 487.2 mm
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Other:
- board size 150 x 142.2 mm -> 150 x 140 mm
- copper layers 4 -> 2
- net class Default: trace_width 0.25 -> 0.3
- net class POWER: trace_width 3.5 -> 3.500001
- rule trace_min: 0.25 -> 0.3
- board text added: "Grzegorz Socha 2022 v.1"
- board text added: "mobile robot motherboard"

Commit message: pre_order
Parts:
- added +BAT: T, TestPoint:TestPoint_Pad_2.5x2.5mm, F.Cu at (43.7, 178.1)
- added 3.3V: T, TestPoint:TestPoint_Pad_2.5x2.5mm, F.Cu at (81.8, 84.2)
- added 5V: T, TestPoint:TestPoint_Pad_2.5x2.5mm, F.Cu at (37.2, 178.1)
- added GND: TestPoint_2Pads_Pitch2.54mm_Drill0.8mm, TestPoint:TestPoint_2Pads_Pitch2.54mm_Drill0.8mm, F.Cu at (71.4, 66.1)
- added REF**: KiCad-Logo_8mm_SilkScreen, Symbol:KiCad-Logo_8mm_SilkScreen, F.Cu at (126.8, 74.3)
- moved REF** 3.45 mm to (34.3, 162.4)
- moved REF** 2.10 mm to (128.9, 65.5)
- moved REF** 1.91 mm to (48.8, 65.5)
- moved REF** 0.82 mm to (152.0, 166.6)
Routing:
- net +5V: track 620.8 -> 631.5 mm
- net +BATT: track 164.4 -> 167.9 mm
- net +3V3: track 487.2 -> 490.3 mm
- net M1INB: track 110.9 -> 107.9 mm
- net M1INA: track 108.2 -> 107.4 mm
- net PA11: track 62.2 -> 61.6 mm
- net GND: vias 251 -> 295
- net BUTTON_2: vias 4 -> 2
- net (no net): vias 3 -> 2
Other:
- board text added: "+"
- board text added: "-"
- board text added: "2022@v1"
- board text added: "Grzegorz Socha https://github.com/IndiaMike"
- board text removed: "Grzegorz Socha 2022 v.1"
